File: board/mainpcb.brd (EAGLE design)
At the start: 141.5 x 25.7 mm, 55 parts, among them IC1 ATMEGA328P, IC2 MAX6921, IC3 7805TV, IC4 DS18B20, J1 2.1MMJACK, Q1 32.768 khz, Q2 IRFD110, SW1 OS102011MA1Q

Commit message: Revised the xmas-icetube board
This commit updates the Ice Tube Clock board to revision C.  Although
revision C is untested, the circuit is identical to revision B, so I
cannot imagine that there would be any problems.
Parts:
- removed DIS1: IV18, vfd:IV18
- removed JP2: male, pinhead:2X10
- D1: value 1N4001 -> MBR160
- D2, D4: value 1N5817 -> MBR160
- F1: value FUSETE5 -> 250 mA
- Q4, Q6: value (none) -> PN2222
- Q5, Q7: value (none) -> PN2907A
- R4: value 10 K -> 5.6 K
- R6: value (none) -> PVD-8001
Connections:
- net VFD'_A renamed VFD'A
- net VFD'_B renamed VFD'B
- net VFD'_C renamed VFD'C
- net VFD'_D renamed VFD'D
- net VFD'_E renamed VFD'E
- net VFD'_F renamed VFD'F
- net VFD'_G renamed VFD'G
- net VFD'_H renamed VFD'H
- removed net AC1': DIS1.1, JP2.11, JP2.12
- removed net AC2': DIS1.13, JP2.2
- removed net VFD1: DIS1.15, JP2.4
- removed net VFD2: DIS1.22, JP2.9
- removed net VFD3: DIS1.16, JP2.3
- removed net VFD4: DIS1.21, JP2.10
- removed net VFD5: DIS1.17, JP2.6
- removed net VFD6: DIS1.20, JP2.7
- removed net VFD7: DIS1.19, JP2.8
- removed net VFD8: DIS1.18, JP2.5
- removed net VFD9: DIS1.14, JP2.1
- removed net VFD_A: DIS1.12, JP2.20
- removed net VFD_B: DIS1.10, JP2.18
- removed net VFD_C: DIS1.4, JP2.15
- removed net VFD_D: DIS1.3, JP2.14
- removed net VFD_E: DIS1.5, JP2.16
- removed net VFD_F: DIS1.11, JP2.19
- removed net VFD_G: DIS1.9, JP2.17
- removed net VFD_H: DIS1.2, JP2.13
Routing:
- net VFD_F: track 29.1 -> 0.00 mm
- net VFD_A: track 28.4 -> 0.00 mm
- net AC2': track 28.3 -> 0.00 mm
- net VFD9: track 28.2 -> 0.00 mm
- net VFD3: track 23.6 -> 0.00 mm
- net VFD_G: track 23.1 -> 0.00 mm
- net VFD_B: track 22.7 -> 0.00 mm
- net VFD1: track 22.0 -> 0.00 mm
- net VFD8: track 18.7 -> 0.00 mm
- net VFD5: track 18.3 -> 0.00 mm
- net VFD6: track 14.3 -> 0.00 mm
- net VFD7: track 12.8 -> 0.00 mm
- net VFD_C: track 12.6 -> 0.00 mm
- net VFD2: track 11.8 -> 0.00 mm
- net AC1': track 11.5 -> 0.00 mm
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- removed copper zone on layer 16, net N$11
- removed copper zone on layer 16, net N$13
- removed copper zone on layer 16, net N$14
- removed copper zone on layer 16, net N$6
- removed copper zone on layer 16, net N$7
- removed copper zone on layer 16, net N$8
Other:
- board size 141.5 x 25.7 mm -> 114.2 x 25.7 mm
- board text added: "BATT"
- board text added: "GND"
- board text added: "J1"
- board text added: "REV C"
- board text added: "RX"
- board text added: "Vreg"
- board text removed: "MERRY"
- board text removed: "REV B"
- board text removed: "XMAS"

Commit message: Revised xmas-icetube board (Rev. D)
The xmas-icetube (Rev D) board is currently *untested*, so use this
design at your own risk.  Rev. D includes an enhancement to the
filament driver circuit to increase filament voltage to within
specifications.  The filament voltage issue has been discussed in the
Adafruit Clocks forum:

  http://forums.adafruit.com/viewtopic.php?p=223798#p223798
  http://forums.adafruit.com/viewtopic.php?p=223793#p223793
Parts:
- added IC5: LM317, jarchie:TO92-LINE
- C6: value 100V/33uF -> 33uF
- D1: value MBR160 -> 1N4001
- D2, D4: value MBR160 -> 1N5817
- D5: value 60V zener -> 56V
- IC3: value 7805TV -> 78L05; device linear:TO220V -> jarchie:TO92-LINE
- Q4, Q6: value PN2222 -> ZVP2110A; device transistor-neu-to92:TO92-EBC -> jarchie:TO92-FLAT
- Q5, Q7: value PN2907A -> ZVN2110A; device transistor-neu-to92:TO92-EBC -> jarchie:TO92-FLAT
- R4: value 5.6 K -> 5.6k
- R5: value 10 K -> 10k
- R7: value 470 -> 1.00k, 1%
- R8: value 470 -> 3.57k, 1%
- moved R8 7.37 mm to (79.1, 12.3), turned to 180 degrees
- moved R6 4.58 mm to (79.4, 2.26)
- moved R7 2.70 mm to (76.6, 8.26), turned to 90 degrees
- moved Q5 2.65 mm to (84.8, 10.0), turned to 270 degrees
- moved Q4 1.69 mm to (84.8, 3.81), turned to 90 degrees
- moved IC3 1.63 mm to (22.9, 24.0), turned to 180 degrees
- moved Q7 1.48 mm to (88.1, 10.0), turned to 270 degrees
- moved Q6 0.54 mm to (88.1, 3.81), turned to 90 degrees
- moved L1 0.25 mm to (71.0, 9.12)
Connections:
- removed net N$10: Q6.B, Q7.B, R8.2
- removed net N$22: Q4.B, Q5.B, R7.2
- new net N$14: IC5.2, Q4.1, Q6.1, R7.1
- new net N$6: IC5.1, R7.2, R8.2
- net +9V: now also IC3.3, IC5.3; no longer IC3.1
- net AC1: now also Q4.3, Q5.3; no longer Q4.E, Q5.E
- net AC1SIG: now also Q4.2, Q5.2; no longer R7.1
- net AC2: now also Q6.3, Q7.3; no longer Q6.E, Q7.E
- net AC2SIG: now also Q6.2, Q7.2; no longer R8.1
- net GND: now also Q5.1, Q7.1, R8.1; no longer Q5.C, Q7.C
- net REGOUT: now also IC3.1; no longer IC3.3
- net VCC: no longer Q4.C, Q6.C
Routing:
- net +9V: track 106.2 -> 189.8 mm
- net VCC: track 181.5 -> 114.8 mm
- net AC2SIG: track 20.3 -> 39.8 mm
- net N$10: track 19.1 -> 0.00 mm
- net GND: track 317.8 -> 336.3 mm
- net N$14: track 0.00 -> 15.2 mm
- net N$22: track 15.0 -> 0.00 mm
- net AC1SIG: track 27.4 -> 39.4 mm
- net N$6: track 0.00 -> 5.43 mm
- net AWAKE: track 43.8 -> 45.6 mm
- net N$2: track 19.0 -> 20.3 mm
- net AC1: track 40.7 -> 39.4 mm
- net REGOUT: track 53.7 -> 54.6 mm
- net AC2: track 31.0 -> 30.4 mm
Other:
- board text added: "REV D"
- board text added: "TOSC1"
- board text removed: "REV C"

Commit message: Minor change to main board.
I changed the main board schematic slightly and added an
acknowledgements section to the README.
Parts:
- C2: value 10uF/25V -> 47uF
Changed lines of the file:
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@@
 <elements>
 <element name="J1" library="minimidi" package="PJ-102A" value="2.1MMJACK" x="12.239" y="25.1206" smashed="yes"/>
-<element name="C2" library="minimidi" package="E2,5-6" value="10uF/25V" x="7.159" y="12.0396" smashed="yes">
+<element name="C2" library="minimidi" package="E2,5-6" value="47uF" x="7.159" y="12.0396" smashed="yes">
 <attribute name="NAME" x="10.207" y="13.3096" size="1.27" layer="25" font="vector" ratio="10" rot="R270"/>
 <attribute name="VALUE" x="9.826" y="9.3726" size="1.27" layer="27" ratio="10"/>

Commit message: Corrected C6 value in board schematic
In both the Ice Tube Clock kit and the xmas-icetube revisions, C6 is
22uF but was marked as 33uF in the schematic.  This has been fixed.
Parts:
- C6: value 33uF -> 22uF
Changed lines of the file:
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@@
 <attribute name="NAME" x="70.118" y="7.1086" size="1.27" layer="21" font="vector"/>
 </element>
-<element name="C6" library="rcl-ez" package="E3,5-8" value="33uF" x="85.518" y="16.8656" smashed="yes" rot="R180">
+<element name="C6" library="rcl-ez" package="E3,5-8" value="22uF" x="85.518" y="16.8656" smashed="yes" rot="R180">
 <attribute name="NAME" x="84.629" y="14.1986" size="1.27" layer="25" font="vector" ratio="10"/>
 <attribute name="VALUE" x="88.82" y="19.9136" size="1.27" layer="27" ratio="10" rot="R180"/>
