File: hardware/mainpcb.brd (EAGLE design)
At the start: 114.2 x 25.7 mm, 54 parts, among them IC1 ATMEGA328P, IC2 MAX6921, IC3 78L05, IC4 DS18B20, IC5 LM317, J1 2.1MMJACK, Q1 32.768 khz, Q2 IRFD110, Q4 ZVP2110A, Q5 ZVN2110A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

Commit message: C6 is now 33uF
Increasing the value of C6 should decrease boost ripple and makes the
schematic consistent with the parts listed in BOM.csv.
Parts:
- C6: value 22uF -> 33uF
Changed lines of the file:
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@@
 <attribute name="NAME" x="70.118" y="7.1086" size="1.27" layer="21" font="vector"/>
 </element>
-<element name="C6" library="rcl-ez" package="E3,5-8" value="22uF" x="85.518" y="16.8656" smashed="yes" rot="R180">
+<element name="C6" library="rcl-ez" package="E3,5-8" value="33uF" x="85.518" y="16.8656" smashed="yes" rot="R180">
 <attribute name="NAME" x="84.629" y="14.1986" size="1.27" layer="25" font="vector" ratio="10"/>
 <attribute name="VALUE" x="88.82" y="19.9136" size="1.27" layer="27" ratio="10" rot="R180"/>
