File: hardware/mainpcb.sch (EAGLE design)
At the start: 54 parts, among them IC1 ATMEGA328P, IC2 MAX6921, IC3 78L05, IC4 DS18B20, IC5 LM317, J1 2.1MMJACK, Q1 32.768 khz, Q2 IRFD110, Q4 ZVP2110A, Q5 ZVN2110A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

Commit message: C6 is now 33uF
Increasing the value of C6 should decrease boost ripple and makes the
schematic consistent with the parts listed in BOM.csv.
Parts:
- C6: value 22uF -> 33uF
Changed lines of the file:
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@@
 <part name="D3" library="usbbuck" deviceset="SCHOTTKY-DIODE" device="DO41" value="MBR160"/>
 <part name="L1" library="usbbuck" deviceset="L" device="" value="2200uH"/>
-<part name="C6" library="rcl-ez" deviceset="CPOL-US" device="E3.5-8" value="22uF"/>
+<part name="C6" library="rcl-ez" deviceset="CPOL-US" device="E3.5-8" value="33uF"/>
 <part name="V2" library="supply2" deviceset="+9V" device=""/>
 <part name="GND3" library="supply1" deviceset="GND" device=""/>
